Commit message: change urdf, replace mat file and delete duplicated files

File: python/urdf/four_joints_two_ft_three_imu.urdf (robot description, URDF)
Before this commit: robot fourjoints, 7 links, 6 joints
Links:
- added link base_imu_0
Joints:
- added joint base_imu_0_fixed_joint: type fixed, parent base_link, child base_imu_0, origin xyz=0.0354497 0.00639688 0.060600 rpy=1.5708 0 -1.5708
- joint joint_1: parent base_link -> base_imu_0
